File: kicad/basic_pid/supply.kicad_sch (KiCad schematic)
At the start: 60 parts, among them J5 Screw_Terminal_01x04, J6 Screw_Terminal_01x03, SW1 SW_DPDT_x2, SW10 SW_DPDT_x2, SW2 SW_DPDT_x2, SW3 SW_DPDT_x2, SW5 SW_DPDT_x2, U14 LM2940CS-12/NOPB, U15 LM2990SX-12, U16 LM317_TO-252

Commit message: version sent to Advanced Circuits and OSHStencils
Connections:
- net V-_unreg: now reaches C19.2, C25.2, D1.4 (-), J6.1 (Pin_1), U15.2 (IN)
- net black: now reaches D1.3, J5.1 (Pin_1)
- net yellow: now reaches D1.2, J5.4 (Pin_4)
Changed lines of the file:
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@@
+    (stroke (width 0) (type default))
+  )
+  (wire (pts (xy 78.105 143.51) (xy 78.105 137.795))
     (stroke (width 0) (type default))
   )
@@
   )
   (wire (pts (xy 175.26 48.895) (xy 175.26 51.435))
+    (stroke (width 0) (type default))
+  )
+  (wire (pts (xy 78.105 143.51) (xy 86.36 143.51))
     (stroke (width 0) (type default))
   )
@@
   (text "Additional parts:\n237-1326-ND VPT30-830 (toroidal transformer)\n	\n1144-1033-ND 06AE2 (Power Entry Module)\n"
     (at 19.05 149.225 0)
+    (effects (font (size 1.27 1.27)) (justify left bottom))
+  )
+  (label "black" (at 36.83 122.555 0) (fields_autoplaced)
+    (effects (font (size 1.27 1.27)) (justify left bottom))
+  )
+  (label "yellow" (at 38.1 141.605 0) (fields_autoplaced)
+    (effects (font (size 1.27 1.27)) (justify left bottom))
+  )
+  (label "red_and_orange" (at 34.925 130.175 0) (fields_autoplaced)
     (effects (font (size 1.27 1.27)) (justify left bottom))
   )
@@
       (effects (font (size 1.27 1.27)) (justify left) hide)
     )
+  )
+  (global_label "V-_unreg" (shape input) (at 86.36 143.51 0) (fields_autoplaced)
+    (effects (font (size 1.27 1.27)) (justify left))
+    (property "Intersheetrefs" "${INTERSHEET_REFS}" (at 98.2162 143.51 0)
+      (effects (font (size 1.27 1.27)) (justify left) hide)
+    )
