File: kicad/smart_pid/basic_pid.kicad_sch (KiCad schematic)
At the start: 36 parts, among them J1 Input A, J2 Input B / Setpoint, J3 Monitor, J4 Output, SW9 SW_SP4T, U12 OPA189, U13 BUF634A, U19 DG419DY-T1-E3, U3 INA849, U4 INA849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

Commit message: Added inverter and modified ext. setpoint disable
Parts:
- removed R42: 10k, Resistor_SMD:R_0805_2012Metric, symbol Device:R_US
- added R29, R62, R63, R64: 10k, Resistor_SMD:R_0805_2012Metric, symbol Device:R_US
- added U2: OPA189, Package_SO:SOIC-8_3.9x4.9mm_P1.27mm, symbol Amplifier_Operational:OPA330xxD
- added U33: DG419DY-T1-E3, Package_SO:SOIC-8_3.9x4.9mm_P1.27mm, symbol Analog_Switch:DG419LDY
Connections:
- net Vlim+ is gone; now on net +12V: U12.7 (V+)
- net Vlim- is gone; now on net -12V: U12.4 (V-)
- net GND: now also U19.8, R62.1
- net IN_B: now also U19.1; no longer U19.2
- net at U4.7: now also U19.2; no longer U19.1
- net D_IN renamed ERR
- net D_OUT renamed D_block/D_OUT
- new net: R63.1, U33.2
- new net: R29.1, U33.8
- new net: R63.2, R64.2, U2.2 (-)
- new net: R29.2, R62.2, U2.3 (+)
- new net: R64.1, U2.6
Other:
- sheet D_block ports: added D_IN, D_OUT; removed none
- moved on the sheet: R6, U19A
