File: kicad/integrator_test/integrator_test/integrator_test.kicad_sch (KiCad schematic)
At the start: 35 parts, among them J1 Conn_01x03_Pin, J2 Conn_01x02_Pin, J3 Conn_01x04_Pin, J4 Conn_01x04_Pin, J5 Conn_01x06_Pin, SW1 SW_SPDT, U19 DG419DY-T1-E3, U23 DG408DQ-T1-E3, U25 MCP45HV51-ST, U9 OPA189

Commit message: integrator test board v2
Parts:
- removed C10, C9: 100nF, Capacitor_SMD:C_0805_2012Metric, symbol Device:C
- removed J1: Conn_01x03_Pin, Connector_PinHeader_2.54mm:PinHeader_1x03_P2.54mm_Vertical, symbol Connector:Conn_01x03_Pin
- removed J2: Conn_01x02_Pin, Connector_PinHeader_2.54mm:PinHeader_1x02_P2.54mm_Vertical, symbol Connector:Conn_01x02_Pin
- removed J5: Conn_01x06_Pin, Connector_PinHeader_2.54mm:PinHeader_1x06_P2.54mm_Vertical, symbol Connector:Conn_01x06_Pin
- removed R17 (x4): 10M, Resistor_SMD:R_0603_1608Metric, symbol Device:R_US
- removed R5: 10k, Resistor_SMD:R_0603_1608Metric, symbol Device:R_US
- removed U25: MCP45HV51-ST, Package_SO:TSSOP-14_4.4x5mm_P0.65mm, symbol Potentiometer_Digital:MCP45HV51-ST
- added C?: DNP, Capacitor_SMD:C_0603_1608Metric, symbol Device:C
- added J3: Conn_01x08_Pin, Connector_PinHeader_2.54mm:PinHeader_1x08_P2.54mm_Vertical, symbol Connector:Conn_01x08_Pin
- added U5: AD5290, Package_SO:MSOP-10_3x3mm_P0.5mm, symbol Potentiometer_Digital:AD5290
- C11, C12, C13, C14, C5, C6, C7, C8: footprint Capacitor_SMD:C_0805_2012Metric -> Capacitor_SMD:C_0603_1608Metric
- C?: renamed from C7; footprint Capacitor_SMD:C_0805_2012Metric -> Capacitor_SMD:C_0603_1608Metric
- C?: renamed from C8; footprint Capacitor_SMD:C_0805_2012Metric -> Capacitor_SMD:C_0603_1608Metric
- C?: renamed from C6; footprint Capacitor_SMD:C_0805_2012Metric -> Capacitor_SMD:C_0603_1608Metric
- C?: renamed from C9; footprint Capacitor_SMD:C_0805_2012Metric -> Capacitor_SMD:C_0603_1608Metric
- renumbered J3 to J1, J4 to J2, R16 to R?, R33 to R?, R34 to R?, R17 to R?, U9 to U?, U23 to U?, U19 to U?
Connections:
- net +12V: now also U5.9 (Vdd+)
- net -12V: now also U5.3 (Vss-)
- net GND: now also U5.4 (GND)
- net INT_CAP_SEL_A0: now also J3.7 (Pin_7)
- net INT_CAP_SEL_A1: now also J3.6 (Pin_6)
- net INT_CAP_SEL_A2: now also J3.5 (Pin_5)
- net INT_R+: now also R6.1, U5.1 (RH)
- net INT_R-: now also C?.1, C?.1, C?.1, C?.1, C?.1, U5.10 (RW); no longer U?.8 (D)
- net I_IN: now also J2.4 (Pin_4); no longer J2.1 (Pin_1)
- net I_OUT: now also J2.1 (Pin_1), U?.8 (D), C?.2; no longer C?.1, C?.1, C?.1, C?.1, J2.4 (Pin_4)
- net I_OVERRIDE_EN: now also J3.8 (Pin_8)
- new net R_CLK: J3.3 (Pin_3), U5.6 (CLK)
- new net R_CS: J3.4 (Pin_4), U5.5 (~{CS})
- new net R_SDI: J3.2 (Pin_2), U5.7 (SDI)
- new net R_SDO: J3.1 (Pin_1), U5.8 (SDO)
- no-connect marks 6 -> 5
Other:
- note added: "Common Mode Leakage: 1000 pA"
- note added: "DG408 - R_on = 100Ω, Source Leakage 500 pA ADG1408 - R_on = 4.7Ω, Source Leakage 200 pA"
- note added: "I_B = 200 pA, I_OS = 120 pA"
- note added: "SDO High: 5V"
- note added: "Source Leakage 250 pA"
- note removed: "DG408 - R_on = 100Ω (ADG1408 - R_on = 4.7Ω)"
- moved on the sheet: C?, U?
